Commit message: Added IMU and Lidar in Gazebo sim with materials

File: src/robot_description/urdf/robot.urdf.xacro (robot description, xacro)
@@ -3,4 +3,5 @@
     <xacro:arg name="is_sim" default="true"/>
     <!-- Include .xacro files -->
+    <xacro:include filename="$(find robot_description)/urdf/materials.xacro"/>
     <xacro:include filename="$(find robot_description)/urdf/robot_gazebo.xacro"/>
     <xacro:include filename="$(find robot_description)/urdf/robot_ros2_control.xacro"/>
@@ -22,4 +23,5 @@
                 <mesh filename="package://robot_description/meshes/base_link.STL"/>
             </geometry>
+            <material name="black"/>
         </visual>
         <collision>
@@ -43,4 +45,5 @@
                 <mesh filename="package://robot_description/meshes/wheel_left_link.STL"/>
             </geometry>
+            <material name="blue"/>
         </visual>
         <collision>
@@ -64,4 +67,5 @@
                 <mesh filename="package://robot_description/meshes/wheel_right_link.STL"/>
             </geometry>
+            <material name="blue"/>
         </visual>
         <collision>
@@ -85,4 +89,5 @@
                 <mesh filename="package://robot_description/meshes/caster_front_link.STL"/>
             </geometry>
+            <material name="silver"/>
         </visual>
         <collision>
@@ -106,4 +111,5 @@
                 <mesh filename="package://robot_description/meshes/caster_rear_link.STL"/>
             </geometry>
+            <material name="silver"/>
         </visual>
         <collision>

File: src/robot_description/urdf/robot_gazebo.xacro (robot description, xacro)
@@ -47,3 +47,84 @@
         </plugin>
     </gazebo>
+    <!-- IMU -->
+    <gazebo reference="imu_link">
+        <sensor name="imu" type="imu">
+            <always_on>true</always_on>
+            <update_rate>100</update_rate>
+            <gz_frame_id>imu_link</gz_frame_id>
+            <topic>imu</topic>
+        </sensor>
+        <imu>
+            <angular_velocity>
+                <x>
+                    <noise type="gaussian">
+                        <mean>0.0</mean>
+                        <stddev>2e-4</stddev>
+                    </noise>
+                </x>
+                <y>
+                    <noise type="gaussian">
+                        <mean>0.0</mean>
+                        <stddev>2e-4</stddev>
+                    </noise>
+                </y>
+                <z>
+                    <noise type="gaussian">
+                        <mean>0.0</mean>
+                        <stddev>2e-4</stddev>
+                    </noise>
+                </z>
+            </angular_velocity>
+            <linear_acceleration>
+                <x>
+                    <noise type="gaussian">
+                        <mean>0.0</mean>
+                        <stddev>1.7e-2</stddev>
+                    </noise>
+                </x>
+                <y>
+                    <noise type="gaussian">
+                        <mean>0.0</mean>
+                        <stddev>1.7e-2</stddev>
+                    </noise>
+                </y>
+                <z>
+                    <noise type="gaussian">
+                        <mean>0.0</mean>
+                        <stddev>1.7e-2</stddev>
+                    </noise>
+                </z>
+            </linear_acceleration>
+        </imu>
+  </gazebo>
+    <!-- Lidar -->
+    <gazebo reference="laser_link">
+        <sensor name="lidar" type="gpu_lidar">
+            <always_on>true</always_on>
+            <visualize>true</visualize>
+            <topic>scan</topic>
+            <update_rate>5</update_rate>
+            <gz_frame_id>laser_link</gz_frame_id>
+            <lidar>
+                <scan>
+                    <horizontal>
+                        <samples>360</samples>
+                        <resolution>1.0</resolution>
+                        <min_angle>0.0</min_angle>
+                        <max_angle>6.28</max_angle>
+                    </horizontal>
+                </scan>
+                <range>
+                    <min>0.12</min>
+                    <max>12.0</max>
+                    <resolution>0.02</resolution>
+                </range>
+                <noise>
+                    <type>gaussian</type>
+                    <mean>0.0</mean>
+                    <stddev>0.01</stddev>
+                </noise>
+            </lidar>
+        </sensor>
+    </gazebo>
 </robot>

File: src/robot_description/urdf/robot_imu.xacro (robot description, xacro)
@@ -3,22 +3,22 @@
     <link name="imu_link">
         <inertial>
-        <origin xyz="-0.00552433659106688 0.000168210391520346 0.000514000497342681" rpy="0 0 0" />
-        <mass value="0.000528415362211671" />
-        <inertia ixx="1.46176048428261E-08" ixy="1.40015117949421E-10" ixz="-1.99633872937403E-12"
-                iyy="8.59662482954888E-09" iyz="7.52375112767959E-12"
-                izz="2.30279421279312E-08" />
+            <origin xyz="-0.00552433659106688 0.000168210391520346 0.000514000497342681" rpy="0 0 0" />
+            <mass value="0.000528415362211671" />
+            <inertia ixx="1.46176048428261E-08" ixy="1.40015117949421E-10" ixz="-1.99633872937403E-12"
+                    iyy="8.59662482954888E-09" iyz="7.52375112767959E-12"
+                    izz="2.30279421279312E-08" />
         </inertial>
         <visual>
-        <origin xyz="0 0 0" rpy="0 0 0"/>
-        <geometry>
-            <mesh filename="package://robot_description/meshes/imu_link.STL"/>
-        </geometry>
-        <material name="blue"/>
+            <origin xyz="0 0 0" rpy="0 0 0"/>
+            <geometry>
+                <mesh filename="package://robot_description/meshes/imu_link.STL"/>
+            </geometry>
+            <material name="blue"/>
         </visual>
         <collision>
-        <origin xyz="0 0 0" rpy="0 0 0"/>
-        <geometry>
-            <mesh filename="package://robot_description/meshes/imu_link.STL"/>
-        </geometry>
+            <origin xyz="0 0 0" rpy="0 0 0"/>
+            <geometry>
+                <mesh filename="package://robot_description/meshes/imu_link.STL"/>
+            </geometry>
         </collision>
     </link>

File: src/robot_description/urdf/robot_lidar.xacro (robot description, xacro)
@@ -14,4 +14,5 @@
                 <mesh filename="package://robot_description/meshes/laser_link.STL"/>
             </geometry>
+            <material name="dark_grey"/>
         </visual>
         <collision>
